File: TNP PCB/TNP Schematic.brd (EAGLE design)
At the start: 67 x 31.7 mm, 5 parts, among them IC1 ULN2003AN, IC2 ULN2003AN

Commit message: Add files via upload
Parts:
- removed JP1, JP2: (no value), pinhead:1X04/90
- added SV1, SV2: (no value), con-lstb:MA05-1
- moved IC1 8.89 mm to (67.3, 67.3), turned to 180 degrees
- moved IC2 7.62 mm to (45.7, 67.3), turned to 180 degrees
Connections:
- net 5V0@1: now also SV2.5
- net 5V0@2: now also SV1.5
- net N$1: now also SV1.1; no longer JP1.1
- net N$2: now also SV1.2; no longer JP1.2
- net N$3: now also SV1.3; no longer JP1.3
- net N$4: now also SV1.4; no longer JP1.4
- net N$5: now also SV2.1; no longer JP2.1
- net N$6: now also SV2.2; no longer JP2.2
- net N$7: now also SV2.3; no longer JP2.3
- net N$8: now also SV2.4; no longer JP2.4
Routing:
- net N$7: track 17.5 -> 68.8 mm
- net N$17: track 85.4 -> 35.0 mm
- net 5V0@1: track 23.3 -> 73.2 mm
- net N$8: track 12.5 -> 51.6 mm
- net GND@8: track 65.8 -> 35.7 mm
- net N$1: track 21.7 -> 5.60 mm
- net N$6: track 21.1 -> 36.1 mm
- net N$12: track 19.4 -> 6.10 mm
- net N$15: track 19.7 -> 32.1 mm
- net 5V0@2: track 45.8 -> 57.7 mm, vias 1 -> 0
- net N$14: track 27.4 -> 17.7 mm
- net N$13: track 19.2 -> 11.2 mm
- net N$2: track 19.9 -> 12.1 mm
- net N$4: track 15.2 -> 23.0 mm
- net N$5: track 23.4 -> 29.3 mm
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