File: TNP PCB/TNP Schematic.sch (EAGLE design)
At the start: 5 parts, among them IC1 ULN2003AN, IC2 ULN2003AN

Commit message: Add files via upload
Parts:
- removed JP1, JP2: (no value), pinhead:PINHD-1X4/90
- added SV1, SV2: (no value), con-lstb:MA05-1
Connections:
- net 5V0@1: now also SV2.5
- net N$1: now also SV1.1; no longer JP1.1
- net N$2: now also SV1.2; no longer JP1.2
- net N$3: now also SV1.3; no longer JP1.3
- net N$4: now also SV1.4; no longer JP1.4
- net N$5: now also SV2.1; no longer JP2.1
- net N$6: now also SV2.2; no longer JP2.2
- net N$7: now also SV2.3; no longer JP2.3
- net N$8: now also SV2.4; no longer JP2.4
Changed lines of the file:
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@@
 <part name="IC1" library="uln-udn" deviceset="ULN2003A" device="N"/>
 <part name="IC2" library="uln-udn" deviceset="ULN2003A" device="N"/>
-<part name="JP1" library="pinhead" deviceset="PINHD-1X4" device="/90"/>
-<part name="JP2" library="pinhead" deviceset="PINHD-1X4" device="/90"/>
+<part name="SV1" library="con-lstb" deviceset="MA05-1" device=""/>
+<part name="SV2" library="con-lstb" deviceset="MA05-1" device=""/>
 </parts>
 <sheets>
@@
 <instance part="IC1" gate="A" x="15.24" y="60.96"/>
 <instance part="IC2" gate="A" x="15.24" y="30.48"/>
-<instance part="JP1" gate="A" x="38.1" y="63.5"/>
-<instance part="JP2" gate="A" x="38.1" y="33.02"/>
+<instance part="SV1" gate="G$1" x="40.64" y="63.5" rot="R180"/>
+<instance part="SV2" gate="G$1" x="40.64" y="33.02" rot="R180"/>
 </instances>
 <busses>
@@
 <net name="N$1" class="0">
 <segment>
-<pinref part="JP1" gate="A" pin="1"/>
+<wire x1="35.56" y1="68.58" x2="33.02" y2="68.58" width="0.1524" layer="91"/>
+<pinref part="SV1" gate="G$1" pin="1"/>
 <pinref part="IC1" gate="A" pin="O1"/>
-<wire x1="35.56" y1="68.58" x2="27.94" y2="68.58" width="0.1524" layer="91"/>
-</segment>
-</net>
-<net name="N$2" class="0">
-<segment>
-<pinref part="JP1" gate="A" pin="2"/>
-<pinref part="IC1" gate="A" pin="O2"/>
-<wire x1="35.56" y1="66.04" x2="27.94" y2="66.04" width="0.1524" layer="91"/>
+<wire x1="27.94" y1="68.58" x2="33.02" y2="68.58" width="0.1524" layer="91"/>
 </segment>
 </net>
 <net name="N$3" class="0">
 <segment>
-<pinref part="JP1" gate="A" pin="3"/>
+<wire x1="35.56" y1="63.5" x2="33.02" y2="63.5" width="0.1524" layer="91"/>
+<pinref part="SV1" gate="G$1" pin="3"/>
 <pinref part="IC1" gate="A" pin="O3"/>
-<wire x1="35.56" y1="63.5" x2="27.94" y2="63.5" width="0.1524" layer="91"/>
+<wire x1="27.94" y1="63.5" x2="33.02" y2="63.5" width="0.1524" layer="91"/>
 </segment>
 </net>
 <net name="N$4" class="0">
 <segment>
+<pinref part="SV1" gate="G$1" pin="4"/>
+<wire x1="33.02" y1="60.96" x2="35.56" y2="60.96" width="0.1524" layer="91"/>
 <pinref part="IC1" gate="A" pin="O4"/>
-<pinref part="JP1" gate="A" pin="4"/>
-<wire x1="27.94" y1="60.96" x2="35.56" y2="60.96" width="0.1524" layer="91"/>
+<wire x1="27.94" y1="60.96" x2="33.02" y2="60.96" width="0.1524" layer="91"/>
 </segment>
 </net>
 <net name="N$5" class="0">
 <segment>
-<pinref part="JP2" gate="A" pin="1"/>
+<wire x1="35.56" y1="38.1" x2="33.02" y2="38.1" width="0.1524" layer="91"/>
+<pinref part="SV2" gate="G$1" pin="1"/>
 <pinref part="IC2" gate="A" pin="O1"/>
-<wire x1="35.56" y1="38.1" x2="27.94" y2="38.1" width="0.1524" layer="91"/>
+<wire x1="27.94" y1="38.1" x2="33.02" y2="38.1" width="0.1524" layer="91"/>
 </segment>
 </net>
 <net name="N$6" class="0">
 <segment>
+<pinref part="SV2" gate="G$1" pin="2"/>
+<wire x1="33.02" y1="35.56" x2="35.56" y2="35.56" width="0.1524" layer="91"/>
 <pinref part="IC2" gate="A" pin="O2"/>
-<pinref part="JP2" gate="A" pin="2"/>
-<wire x1="27.94" y1="35.56" x2="35.56" y2="35.56" width="0.1524" layer="91"/>
+<wire x1="27.94" y1="35.56" x2="33.02" y2="35.56" width="0.1524" layer="91"/>
 </segment>
 </net>
 <net name="N$7" class="0">
 <segment>
-<pinref part="JP2" gate="A" pin="3"/>
+<wire x1="35.56" y1="33.02" x2="33.02" y2="33.02" width="0.1524" layer="91"/>
+<pinref part="SV2" gate="G$1" pin="3"/>
 <pinref part="IC2" gate="A" pin="O3"/>
-<wire x1="35.56" y1="33.02" x2="27.94" y2="33.02" width="0.1524" layer="91"/>
+<wire x1="27.94" y1="33.02" x2="33.02" y2="33.02" width="0.1524" layer="91"/>
 </segment>
 </net>
 <net name="N$8" class="0">
 <segment>
-<pinref part="JP2" gate="A" pin="4"/>
+<wire x1="35.56" y1="30.48" x2="33.02" y2="30.48" width="0.1524" layer="91"/>
+<pinref part="SV2" gate="G$1" pin="4"/>
 <pinref part="IC2" gate="A" pin="O4"/>
-<wire x1="35.56" y1="30.48" x2="27.94" y2="30.48" width="0.1524" layer="91"/>
+<wire x1="27.94" y1="30.48" x2="33.02" y2="30.48" width="0.1524" layer="91"/>
 </segment>
 </net>
@@
 <segment>
 <pinref part="IC2" gate="A" pin="CD+"/>
-<wire x1="27.94" y1="20.32" x2="45.72" y2="20.32" width="0.1524" layer="91"/>
+<wire x1="27.94" y1="20.32" x2="33.02" y2="20.32" width="0.1524" layer="91"/>
+<wire x1="33.02" y1="20.32" x2="45.72" y2="20.32" width="0.1524" layer="91"/>
 <wire x1="45.72" y1="20.32" x2="45.72" y2="73.66" width="0.1524" layer="91"/>
 <pinref part="U$1" gate="G$1" pin="5V0@1"/>
 <wire x1="45.72" y1="73.66" x2="109.22" y2="73.66" width="0.1524" layer="91"/>
 <wire x1="109.22" y1="73.66" x2="109.22" y2="68.58" width="0.1524" layer="91"/>
+<pinref part="SV2" gate="G$1" pin="5"/>
+<wire x1="33.02" y1="27.94" x2="33.02" y2="20.32" width="0.1524" layer="91"/>
+<wire x1="33.02" y1="27.94" x2="35.56" y2="27.94" width="0.1524" layer="91"/>
 </segment>
 </net>
@@
 <segment>
 <pinref part="IC1" gate="A" pin="CD+"/>
-<wire x1="27.94" y1="50.8" x2="43.18" y2="50.8" width="0.1524" layer="91"/>
+<wire x1="27.94" y1="50.8" x2="33.02" y2="50.8" width="0.1524" layer="91"/>
+<wire x1="33.02" y1="50.8" x2="43.18" y2="50.8" width="0.1524" layer="91"/>
 <wire x1="43.18" y1="50.8" x2="43.18" y2="76.2" width="0.1524" layer="91"/>
 <wire x1="43.18" y1="76.2" x2="111.76" y2="76.2" width="0.1524" layer="91"/>
@@
 <pinref part="U$1" gate="G$1" pin="5V0@2"/>
 <wire x1="111.76" y1="66.04" x2="109.22" y2="66.04" width="0.1524" layer="91"/>
+<wire x1="35.56" y1="58.42" x2="33.02" y2="58.42" width="0.1524" layer="91"/>
+<wire x1="33.02" y1="58.42" x2="33.02" y2="50.8" width="0.1524" layer="91"/>
 </segment>
 </net>
@@
 </segment>
 </net>
+<net name="N$2" class="0">
+<segment>
+<pinref part="IC1" gate="A" pin="O2"/>
+<pinref part="SV1" gate="G$1" pin="2"/>
+<wire x1="27.94" y1="66.04" x2="33.02" y2="66.04" width="0.1524" layer="91"/>
+</segment>
+</net>
